Commit message: fix: metapackage, naming

File: src/zed_description/urdf/zed2i.urdf.xacro (robot description, xacro)
@@ -1,5 +1,6 @@
 <?xml version="1.0"?>
 <robot xmlns:xacro="http://ros.org/wiki/xacro"
-       xmlns:ignition="http://ignitionrobotics.org/schema" name="zed">
+       xmlns:ignition="http://ignitionrobotics.org/schema"
+       name="zed2i">
   <!-- ZED2i -->
   <xacro:property name="zed2i_z" value = "0.0373"/>
@@ -9,5 +10,5 @@
   <xacro:property name="zed2i_imu_to_left_z" value = "-0.00022"/>
   <!-- Function -->
-  <xacro:macro name="zed">
+  <xacro:macro name="zed2i">
     <!-- ZED2i -->
     <link name="zed2i_center_link"></link>

Commit message: fix: remove minus sign from zed urdf

File: src/zed_description/urdf/zed2i.urdf.xacro (robot description, xacro)
@@ -8,5 +8,5 @@
   <xacro:property name="zed2i_imu_to_left_x" value = "0.002"/>
   <xacro:property name="zed2i_imu_to_left_y" value = "0.023"/>
-  <xacro:property name="zed2i_imu_to_left_z" value = "-0.00022"/>
+  <xacro:property name="zed2i_imu_to_left_z" value = "0.00022"/>
   <!-- Function -->
   <xacro:macro name="zed2i">
@@ -16,5 +16,5 @@
       <parent link="base_link"/>
       <child link="zed2i_center_link"/>
-      <origin rpy="0 -${zed2i_tilt} 0" xyz="${zed2i_to_base_link_x} ${zed2i_to_base_link_y} ${zed2i_to_base_link_z}"/>
+      <origin rpy="0 ${zed2i_tilt} 0" xyz="${zed2i_to_base_link_x} ${zed2i_to_base_link_y} ${zed2i_to_base_link_z}"/>
     </joint>
     <link name="zed2i_right_link"></link>
